Commit message: New URDF

File: description/robot.body.xacro (robot description, xacro)
@@ -43,4 +43,7 @@
         </xacro:inertial_box>
     </link>
+    <gazebo reference="chassis">
+        <material>Gazebo/white</material>
+    </gazebo>
     <!-- Front Left Wheel -->
     <joint name="front_left_wheel_joint" type="continuous">
@@ -66,4 +69,7 @@
         </xacro:inertial_cylinder>
     </link>
+    <gazebo reference="front_left_wheel">
+        <material>Gazebo/Black</material>
+    </gazebo>
     <!-- Front Right Wheel -->
     <joint name="front_right_wheel_joint" type="continuous">
@@ -89,4 +95,7 @@
         </xacro:inertial_cylinder>
     </link>
+    <gazebo reference="front_right_wheel">
+        <material>Gazebo/Black</material>
+    </gazebo>
     <!-- Rear Left Wheel -->
     <joint name="rear_left_wheel_joint" type="continuous">
@@ -112,4 +121,7 @@
         </xacro:inertial_cylinder>
     </link>
+    <gazebo reference="rear_left_wheel">
+        <material>Gazebo/Black</material>
+    </gazebo>
     <!-- Rear Right Wheel -->
     <joint name="rear_right_wheel_joint" type="continuous">
@@ -135,3 +147,6 @@
         </xacro:inertial_cylinder>
     </link>
+        <gazebo reference="rear_right_wheel">
+        <material>Gazebo/Black</material>
+    </gazebo>
 </robot>

Commit message: Nuevo URDF

File: description/robot.body.xacro (robot description, xacro)
@@ -2,4 +2,5 @@
 <robot xmlns:xacro="http://www.ros.org/wiki/xacro">
     <xacro:include filename="inertial.macros.xacro"/>
+    <!-- Materials -->
     <material name="white">
         <color rgba="1 1 1 1" />
@@ -17,4 +18,5 @@
         <color rgba="1 0 0 1"/>
     </material>
+    <!-- Base Link -->
     <link name="base_link">
     </link>
@@ -40,30 +42,69 @@
         </collision>
         <xacro:inertial_box mass="0.5" x="0.5" y="0.3" z="0.15">
-        <origin xyz="0.15 0 0.075" rpy="0 0 0"/>
+            <origin xyz="0.15 0 0.075" rpy="0 0 0"/>
         </xacro:inertial_box>
     </link>
     <gazebo reference="chassis">
-        <material>Gazebo/white</material>
-    </gazebo>
+        <material>Gazebo/White</material>
+    </gazebo>
+    <!-- Front Left Steering Joint -->
+    <joint name="front_left_steering_joint" type="revolute">
+        <parent link="base_link"/>
+        <child link="front_left_steering"/>
+        <origin xyz="0.15 0.175 0" rpy="0 0 0"/>
+        <axis xyz="0 0 1"/>
+        <limit lower="-0.8" upper="0.8" effort="10" velocity="5"/>
+    </joint>
+    <link name="front_left_steering">
+        <visual>
+            <geometry>
+                <cylinder radius="0.01" length="0.05"/>
+            </geometry>
+            <material name="red"/>
+        </visual>
+        <xacro:inertial_cylinder mass="0.01" length="0.05" radius="0.01">
+            <origin xyz="0 0 0" rpy="0 0 0"/>
+        </xacro:inertial_cylinder>
+    </link>
+    <!-- Front Right Steering Joint -->
+    <joint name="front_right_steering_joint" type="revolute">
+        <parent link="base_link"/>
+        <child link="front_right_steering"/>
+        <origin xyz="0.15 -0.175 0" rpy="0 0 0"/>
+        <axis xyz="0 0 1"/>
+        <limit lower="-0.8" upper="0.8" effort="10" velocity="5"/>
+    </joint>
+    <link name="front_right_steering">
+        <visual>
+            <geometry>
+                <cylinder radius="0.01" length="0.05"/>
+            </geometry>
+            <material name="red"/>
+        </visual>
+        <xacro:inertial_cylinder mass="0.01" length="0.05" radius="0.01">
+            <origin xyz="0 0 0" rpy="0 0 0"/>
+        </xacro:inertial_cylinder>
+    </link>
     <!-- Front Left Wheel -->
-    <joint name="front_left_wheel_joint" type="continuous">
-        <parent link="base_link"/>
+    <joint name="front_left_wheel_joint" type="revolute">
+        <parent link="front_left_steering"/>
         <child link="front_left_wheel"/>
-        <origin xyz="0.15 0.175 0" rpy="-${pi/2} 0 0"/>
-        <axis xyz="0 0 1"/>
+        <origin xyz="0 0 0" rpy="-${pi/2} 0 0"/>
+        <axis xyz="0 0 1"/>
+        <limit lower="-0.8" upper="0.8" effort="10" velocity="5"/>
     </joint>
     <link name="front_left_wheel">
         <visual>
             <geometry>
-                <cylinder radius="0.05" length="0.04"/>
-            </geometry>
-            <material name="blue"/>
-        </visual>
-        <collision>
-            <geometry>
-                <cylinder radius="0.05" length="0.04"/>
-            </geometry>
-        </collision>
-        <xacro:inertial_cylinder mass="0.1" length="0.04" radius="0.5">
+                <cylinder radius="0.1" length="0.04"/>
+            </geometry>
+            <material name="blue"/>
+        </visual>
+        <collision>
+            <geometry>
+                <cylinder radius="0.1" length="0.04"/>
+            </geometry>
+        </collision>
+        <xacro:inertial_cylinder mass="0.1" length="0.04" radius="0.1">
             <origin xyz="0 0 0" rpy="0 0 0"/>
         </xacro:inertial_cylinder>
@@ -71,25 +112,28 @@
     <gazebo reference="front_left_wheel">
         <material>Gazebo/Black</material>
+        <mu1 value="0.001"/>
+        <mu2 value="0.001"/>
     </gazebo>
     <!-- Front Right Wheel -->
-    <joint name="front_right_wheel_joint" type="continuous">
-        <parent link="base_link"/>
+    <joint name="front_right_wheel_joint" type="revolute">
+        <parent link="front_right_steering"/>
         <child link="front_right_wheel"/>
-        <origin xyz="0.15 -0.175 0" rpy="${pi/2} 0 0"/>
-        <axis xyz="0 0 -1"/>
+        <origin xyz="0 0 0" rpy="${pi/2} 0 0"/>
+        <axis xyz="0 0 1"/>
+        <limit lower="-0.8" upper="0.8" effort="10" velocity="5"/>
     </joint>
     <link name="front_right_wheel">
         <visual>
             <geometry>
-                <cylinder radius="0.05" length="0.04"/>
-            </geometry>
-            <material name="blue"/>
-        </visual>
-        <collision>
-            <geometry>
-                <cylinder radius="0.05" length="0.04"/>
-            </geometry>
-        </collision>
-        <xacro:inertial_cylinder mass="0.1" length="0.04" radius="0.5">
+                <cylinder radius="0.1" length="0.04"/>
+            </geometry>
+            <material name="blue"/>
+        </visual>
+        <collision>
+            <geometry>
+                <cylinder radius="0.1" length="0.04"/>
+            </geometry>
+        </collision>
+        <xacro:inertial_cylinder mass="0.1" length="0.04" radius="0.1">
             <origin xyz="0 0 0" rpy="0 0 0"/>
         </xacro:inertial_cylinder>
@@ -97,25 +141,28 @@
     <gazebo reference="front_right_wheel">
         <material>Gazebo/Black</material>
+        <mu1 value="0.001"/>
+        <mu2 value="0.001"/>
     </gazebo>
     <!-- Rear Left Wheel -->
-    <joint name="rear_left_wheel_joint" type="continuous">
+    <joint name="rear_left_wheel_joint" type="revolute">
         <parent link="base_link"/>
         <child link="rear_left_wheel"/>
         <origin xyz="-0.15 0.175 0" rpy="-${pi/2} 0 0"/>
         <axis xyz="0 0 1"/>
+        <limit lower="-0.8" upper="0.8" effort="10" velocity="5"/>
     </joint>
     <link name="rear_left_wheel">
         <visual>
             <geometry>
-                <cylinder radius="0.05" length="0.04"/>
-            </geometry>
-            <material name="blue"/>
-        </visual>
-        <collision>
-            <geometry>
-                <cylinder radius="0.05" length="0.04"/>
-            </geometry>
-        </collision>
-        <xacro:inertial_cylinder mass="0.1" length="0.04" radius="0.5">
+                <cylinder radius="0.1" length="0.04"/>
+            </geometry>
+            <material name="blue"/>
+        </visual>
+        <collision>
+            <geometry>
+                <cylinder radius="0.1" length="0.04"/>
+            </geometry>
+        </collision>
+        <xacro:inertial_cylinder mass="0.1" length="0.04" radius="0.1">
             <origin xyz="0 0 0" rpy="0 0 0"/>
         </xacro:inertial_cylinder>
@@ -125,27 +172,28 @@
     </gazebo>
     <!-- Rear Right Wheel -->
-    <joint name="rear_right_wheel_joint" type="continuous">
+    <joint name="rear_right_wheel_joint" type="revolute">
         <parent link="base_link"/>
         <child link="rear_right_wheel"/>
         <origin xyz="-0.15 -0.175 0" rpy="${pi/2} 0 0"/>
-        <axis xyz="0 0 -1"/>
+        <axis xyz="0 0 1"/>
+        <limit lower="-0.8" upper="0.8" effort="10" velocity="5"/>
     </joint>
     <link name="rear_right_wheel">
         <visual>
             <geometry>
-                <cylinder radius="0.05" length="0.04"/>
-            </geometry>
-            <material name="blue"/>
-        </visual>
-        <collision>
-            <geometry>
-                <cylinder radius="0.05" length="0.04"/>
-            </geometry>
-        </collision>
-        <xacro:inertial_cylinder mass="0.1" length="0.04" radius="0.5">
-            <origin xyz="0 0 0" rpy="0 0 0"/>
-        </xacro:inertial_cylinder>
-    </link>
-        <gazebo reference="rear_right_wheel">
+                <cylinder radius="0.1" length="0.04"/>
+            </geometry>
+            <material name="blue"/>
+        </visual>
+        <collision>
+            <geometry>
+                <cylinder radius="0.1" length="0.04"/>
+            </geometry>
+        </collision>
+        <xacro:inertial_cylinder mass="0.1" length="0.04" radius="0.1">
+            <origin xyz="0 0 0" rpy="0 0 0"/>
+        </xacro:inertial_cylinder>
+    </link>
+    <gazebo reference="rear_right_wheel">
         <material>Gazebo/Black</material>
     </gazebo>

File: description/robot.urdf.xacro (robot description, xacro)
@@ -2,3 +2,4 @@
 <robot xmlns:xacro="http://www.ros.org/wiki/xacro"  name="robot">
     <xacro:include filename="robot.body.xacro" />
+    <xacro:include filename="gazebo.control.xacro"/>
 </robot>

Commit message: Nuevo URDF

File: description/robot.body.xacro (robot description, xacro)
@@ -48,49 +48,10 @@
         <material>Gazebo/White</material>
     </gazebo>
-    <!-- Front Left Steering Joint -->
-    <joint name="front_left_steering_joint" type="revolute">
-        <parent link="base_link"/>
-        <child link="front_left_steering"/>
-        <origin xyz="0.15 0.175 0" rpy="0 0 0"/>
-        <axis xyz="0 0 1"/>
-        <limit lower="-0.8" upper="0.8" effort="10" velocity="5"/>
-    </joint>
-    <link name="front_left_steering">
-        <visual>
-            <geometry>
-                <cylinder radius="0.01" length="0.05"/>
-            </geometry>
-            <material name="red"/>
-        </visual>
-        <xacro:inertial_cylinder mass="0.01" length="0.05" radius="0.01">
-            <origin xyz="0 0 0" rpy="0 0 0"/>
-        </xacro:inertial_cylinder>
-    </link>
-    <!-- Front Right Steering Joint -->
-    <joint name="front_right_steering_joint" type="revolute">
-        <parent link="base_link"/>
-        <child link="front_right_steering"/>
-        <origin xyz="0.15 -0.175 0" rpy="0 0 0"/>
-        <axis xyz="0 0 1"/>
-        <limit lower="-0.8" upper="0.8" effort="10" velocity="5"/>
-    </joint>
-    <link name="front_right_steering">
-        <visual>
-            <geometry>
-                <cylinder radius="0.01" length="0.05"/>
-            </geometry>
-            <material name="red"/>
-        </visual>
-        <xacro:inertial_cylinder mass="0.01" length="0.05" radius="0.01">
-            <origin xyz="0 0 0" rpy="0 0 0"/>
-        </xacro:inertial_cylinder>
-    </link>
     <!-- Front Left Wheel -->
-    <joint name="front_left_wheel_joint" type="revolute">
-        <parent link="front_left_steering"/>
+    <joint name="front_left_wheel_joint" type="continuous">
+        <parent link="chassis"/>
         <child link="front_left_wheel"/>
         <origin xyz="0 0 0" rpy="-${pi/2} 0 0"/>
         <axis xyz="0 0 1"/>
-        <limit lower="-0.8" upper="0.8" effort="10" velocity="5"/>
     </joint>
     <link name="front_left_wheel">
@@ -116,10 +77,9 @@
     </gazebo>
     <!-- Front Right Wheel -->
-    <joint name="front_right_wheel_joint" type="revolute">
-        <parent link="front_right_steering"/>
+    <joint name="front_right_wheel_joint" type="continuous">
+        <parent link="chassis"/>
         <child link="front_right_wheel"/>
         <origin xyz="0 0 0" rpy="${pi/2} 0 0"/>
-        <axis xyz="0 0 1"/>
-        <limit lower="-0.8" upper="0.8" effort="10" velocity="5"/>
+        <axis xyz="0 0 -1"/>
     </joint>
     <link name="front_right_wheel">
@@ -145,10 +105,9 @@
     </gazebo>
     <!-- Rear Left Wheel -->
-    <joint name="rear_left_wheel_joint" type="revolute">
-        <parent link="base_link"/>
+    <joint name="rear_left_wheel_joint" type="continuous">
+        <parent link="chassis"/>
         <child link="rear_left_wheel"/>
         <origin xyz="-0.15 0.175 0" rpy="-${pi/2} 0 0"/>
         <axis xyz="0 0 1"/>
-        <limit lower="-0.8" upper="0.8" effort="10" velocity="5"/>
     </joint>
     <link name="rear_left_wheel">
@@ -172,10 +131,9 @@
     </gazebo>
     <!-- Rear Right Wheel -->
-    <joint name="rear_right_wheel_joint" type="revolute">
-        <parent link="base_link"/>
+    <joint name="rear_right_wheel_joint" type="continuous">
+        <parent link="chassis"/>
         <child link="rear_right_wheel"/>
         <origin xyz="-0.15 -0.175 0" rpy="${pi/2} 0 0"/>
-        <axis xyz="0 0 1"/>
-        <limit lower="-0.8" upper="0.8" effort="10" velocity="5"/>
+        <axis xyz="0 0 -1"/>
     </joint>
     <link name="rear_right_wheel">

Commit message: Nuevo URDF

File: description/robot.body.xacro (robot description, xacro)
@@ -52,5 +52,5 @@
         <parent link="chassis"/>
         <child link="front_left_wheel"/>
-        <origin xyz="0 0 0" rpy="-${pi/2} 0 0"/>
+        <origin xyz="0.15 0.175 0" rpy="-${pi/2} 0 0"/>
         <axis xyz="0 0 1"/>
     </joint>
@@ -78,5 +78,5 @@
         <parent link="chassis"/>
         <child link="front_right_wheel"/>
-        <origin xyz="0 0 0" rpy="${pi/2} 0 0"/>
+        <origin xyz="0.15 -0.175 0" rpy="${pi/2} 0 0"/>
         <axis xyz="0 0 -1"/>
     </joint>

Commit message: New URDF

File: description/robot.body.xacro (robot description, xacro)
@@ -52,5 +52,5 @@
         <parent link="chassis"/>
         <child link="front_left_wheel"/>
-        <origin xyz="0.15 0.175 0" rpy="-${pi/2} 0 0"/>
+        <origin xyz="0.15 0.175 0.15" rpy="-${pi/2} 0 0"/>
         <axis xyz="0 0 1"/>
     </joint>
@@ -78,5 +78,5 @@
         <parent link="chassis"/>
         <child link="front_right_wheel"/>
-        <origin xyz="0.15 -0.175 0" rpy="${pi/2} 0 0"/>
+        <origin xyz="0.15 -0.175 0.15" rpy="${pi/2} 0 0"/>
         <axis xyz="0 0 -1"/>
     </joint>
@@ -104,5 +104,5 @@
         <parent link="chassis"/>
         <child link="rear_left_wheel"/>
-        <origin xyz="-0.15 0.175 0" rpy="-${pi/2} 0 0"/>
+        <origin xyz="-0.15 0.175 0.15" rpy="-${pi/2} 0 0"/>
         <axis xyz="0 0 1"/>
     </joint>
@@ -130,5 +130,5 @@
         <parent link="chassis"/>
         <child link="rear_right_wheel"/>
-        <origin xyz="-0.15 -0.175 0" rpy="${pi/2} 0 0"/>
+        <origin xyz="-0.15 -0.175 0.15" rpy="${pi/2} 0 0"/>
         <axis xyz="0 0 -1"/>
     </joint>

Commit message: Nuevo URDF

File: description/robot.body.xacro (robot description, xacro)
@@ -52,5 +52,5 @@
         <parent link="chassis"/>
         <child link="front_left_wheel"/>
-        <origin xyz="0.15 0.175 0.15" rpy="-${pi/2} 0 0"/>
+        <origin xyz="0.29 0.175 0" rpy="-${pi/2} 0 0"/>
         <axis xyz="0 0 1"/>
     </joint>
@@ -78,5 +78,5 @@
         <parent link="chassis"/>
         <child link="front_right_wheel"/>
-        <origin xyz="0.15 -0.175 0.15" rpy="${pi/2} 0 0"/>
+        <origin xyz="0.29 -0.175 0" rpy="${pi/2} 0 0"/>
         <axis xyz="0 0 -1"/>
     </joint>
@@ -102,7 +102,7 @@
     <!-- Rear Left Wheel -->
     <joint name="rear_left_wheel_joint" type="continuous">
-        <parent link="chassis"/>
+        <parent link="base_link"/>
         <child link="rear_left_wheel"/>
-        <origin xyz="-0.15 0.175 0.15" rpy="-${pi/2} 0 0"/>
+        <origin xyz="-0.15 0.175 0" rpy="-${pi/2} 0 0"/>
         <axis xyz="0 0 1"/>
     </joint>
@@ -128,7 +128,7 @@
     <!-- Rear Right Wheel -->
     <joint name="rear_right_wheel_joint" type="continuous">
-        <parent link="chassis"/>
+        <parent link="base_link"/>
         <child link="rear_right_wheel"/>
-        <origin xyz="-0.15 -0.175 0.15" rpy="${pi/2} 0 0"/>
+        <origin xyz="-0.15 -0.175 0" rpy="${pi/2} 0 0"/>
         <axis xyz="0 0 -1"/>
     </joint>

Commit message: Nuevo URDF

File: description/robot.body.xacro (robot description, xacro)
@@ -81,5 +81,5 @@
         <child link="front_right_wheel"/>
         <origin xyz="0.29 -0.175 0" rpy="${pi/2} 0 0"/>
-        <axis xyz="0 0 -1"/>
+        <axis xyz="0 0 1"/>
     </joint>
     <link name="front_right_wheel">
@@ -106,7 +106,7 @@
     <!-- Rear Left Wheel -->
     <joint name="rear_left_wheel_joint" type="continuous">
-        <parent link="chassis"/>
+        <parent link="base_link"/>
         <child link="rear_left_wheel"/>
-        <origin xyz="-0.04 0.175 0" rpy="-${pi/2} 0 0"/>
+        <origin xyz="-0.15 0.175 0" rpy="-${pi/2} 0 0"/>
         <axis xyz="0 0 1"/>
     </joint>
@@ -132,8 +132,8 @@
     <!-- Rear Right Wheel -->
     <joint name="rear_right_wheel_joint" type="continuous">
-        <parent link="chassis"/>
+        <parent link="base_link"/>
         <child link="rear_right_wheel"/>
-        <origin xyz="-0.04 -0.175 0" rpy="${pi/2} 0 0"/>
-        <axis xyz="0 0 -1"/>
+        <origin xyz="-0.15 -0.175 0" rpy="${pi/2} 0 0"/>
+        <axis xyz="0 0 1"/>
     </joint>
     <link name="rear_right_wheel">

Commit message: 4W working

File: description/robot.body.xacro (robot description, xacro)
@@ -80,5 +80,5 @@
         <parent link="base_link"/>
         <child link="front_right_wheel"/>
-        <origin xyz="0.2 -0.175 0" rpy="${pi/2} 0 0"/>
+        <origin xyz="0.2 -0.175 0" rpy="-${pi/2} 0 0"/>
         <axis xyz="0 0 1"/>
     </joint>
@@ -134,5 +134,5 @@
         <parent link="base_link"/>
         <child link="rear_right_wheel"/>
-        <origin xyz="-0.2 -0.175 0" rpy="${pi/2} 0 0"/>
+        <origin xyz="-0.2 -0.175 0" rpy="-${pi/2} 0 0"/>
         <axis xyz="0 0 1"/>
     </joint>

Commit message: Changes

File: description/robot.body.xacro (robot description, xacro)
@@ -52,5 +52,5 @@
         <parent link="base_link"/>
         <child link="front_left_wheel"/>
-        <origin xyz="0.2 0.175 0" rpy="-${pi/2} 0 0"/>
+        <origin xyz="0.2 0.175 0" rpy="${pi/2} 0 0"/>
         <axis xyz="0 0 1"/>
     </joint>

Commit message: 4 Wheels functioning

File: description/robot.body.xacro (robot description, xacro)
@@ -52,5 +52,5 @@
         <parent link="base_link"/>
         <child link="front_left_wheel"/>
-        <origin xyz="0.2 0.175 0" rpy="${pi/2} 0 0"/>
+        <origin xyz="0.2 0.175 0" rpy="-${pi/2} 0 0"/>
         <axis xyz="0 0 1"/>
     </joint>
@@ -80,6 +80,6 @@
         <parent link="base_link"/>
         <child link="front_right_wheel"/>
-        <origin xyz="0.2 -0.175 0" rpy="-${pi/2} 0 0"/>
-        <axis xyz="0 0 1"/>
+        <origin xyz="0.2 -0.175 0" rpy="${pi/2} 0 0"/>
+        <axis xyz="0 0 -1"/>
     </joint>
     <link name="front_right_wheel">
@@ -134,6 +134,6 @@
         <parent link="base_link"/>
         <child link="rear_right_wheel"/>
-        <origin xyz="-0.2 -0.175 0" rpy="-${pi/2} 0 0"/>
-        <axis xyz="0 0 1"/>
+        <origin xyz="-0.2 -0.175 0" rpy="${pi/2} 0 0"/>
+        <axis xyz="0 0 -1"/>
     </joint>
     <link name="rear_right_wheel">
