Commit message: NUevo URDF

File: description/gazebo.control.xacro (robot description, xacro)
@@ -3,13 +3,12 @@
     <gazebo>
         <plugin name="diff_drive" filename="libgazebo_ros_diff_drive.so">
-            <!-- Wheel Information -->
-            <left_joint>rear_left_wheel_joint</left_joint>
             <left_joint>front_left_wheel_joint</left_joint>
+            <left_joint>front_left_wheel_joint</left_joint>
+            <right_joint>rear_right_wheel_joint</right_joint>
+            <right_joint>front_right_wheel_joint</right_joint>
             <wheel_separation>0.35</wheel_separation>
             <wheel_diameter>0.1</wheel_diameter>
-            <!-- Limits -->
             <max_wheel_torque>200</max_wheel_torque>
             <max_wheel_acceleration>10.0</max_wheel_acceleration>
-            <!-- Output -->
             <odometry_frame>odom</odometry_frame>
             <robot_base_frame>base_link</robot_base_frame>
@@ -17,4 +16,5 @@
             <publish_odom_tf>true</publish_odom_tf>
             <publish_wheel_tf>true</publish_wheel_tf>
+            <command_topic>cdm_vel</command_topic>
         </plugin>
     </gazebo>

File: description/robot.body.xacro (robot description, xacro)
@@ -106,7 +106,7 @@
     <!-- Rear Left Wheel -->
     <joint name="rear_left_wheel_joint" type="continuous">
-        <parent link="base_link"/>
+        <parent link="chassis"/>
         <child link="rear_left_wheel"/>
-        <origin xyz="-0.15 0.175 0" rpy="-${pi/2} 0 0"/>
+        <origin xyz="-0.04 0.175 0" rpy="-${pi/2} 0 0"/>
         <axis xyz="0 0 1"/>
     </joint>
@@ -132,7 +132,7 @@
     <!-- Rear Right Wheel -->
     <joint name="rear_right_wheel_joint" type="continuous">
-        <parent link="base_link"/>
+        <parent link="chassis"/>
         <child link="rear_right_wheel"/>
-        <origin xyz="-0.15 -0.175 0" rpy="${pi/2} 0 0"/>
+        <origin xyz="-0.04 -0.175 0" rpy="${pi/2} 0 0"/>
         <axis xyz="0 0 -1"/>
     </joint>

Commit message: New URDF

File: description/gazebo.control.xacro (robot description, xacro)
@@ -2,13 +2,29 @@
 <robot xmlns:xacro="http://www.ros.org/wiki/xacro">
     <gazebo>
-        <plugin name="diff_drive" filename="libgazebo_ros_diff_drive.so">
+        <plugin name="front_wheel" filename="libgazebo_ros_diff_drive.so">
         <!-- Wheels-->
             <left_joint>front_left_wheel_joint</left_joint>
-            <left_joint>front_left_wheel_joint</left_joint>
-            <right_joint>rear_right_wheel_joint</right_joint>
-            <right_joint>front_right_wheel_joint</right_joint>
+            <left_joint>front_right_wheel_joint</left_joint>
             <wheel_separation>0.35</wheel_separation>
             <wheel_diameter>0.1</wheel_diameter>
-        <!-- Limtirs-->
+        <!-- Limtis-->
+            <max_wheel_torque>200</max_wheel_torque>
+            <max_wheel_acceleration>10.0</max_wheel_acceleration>
+        <!-- Output-->
+            <odometry_frame>odom</odometry_frame>
+            <robot_base_frame>base_link</robot_base_frame>
+            <publish_odom>true</publish_odom>
+            <publish_odom_tf>true</publish_odom_tf>
+            <publish_wheel_tf>true</publish_wheel_tf>
+        </plugin>
+    </gazebo>
+    <gazebo>
+        <plugin name="rear_wheel" filename="libgazebo_ros_diff_drive.so">
+        <!-- Wheels-->
+            <left_joint>rear_left_wheel_joint</left_joint>
+            <left_joint>rear_right_wheel_joint</left_joint>
+            <wheel_separation>0.35</wheel_separation>
+            <wheel_diameter>0.1</wheel_diameter>
+        <!-- Limtis-->
             <max_wheel_torque>200</max_wheel_torque>
             <max_wheel_acceleration>10.0</max_wheel_acceleration>

File: description/inertial.macros.xacro (robot description, xacro)
@@ -21,3 +21,12 @@
         </inertial>
     </xacro:macro>
+    <xacro:macro name="inertial_sphere" params="mass radius *origin">
+        <inertial>
+            <xacro:insert_block name="origin"/>
+            <mass value="${mass}" />
+            <inertia ixx="${(2/5) * mass * (radius*radius)}" ixy="0.0" ixz="0.0"
+                    iyy="${(2/5) * mass * (radius*radius)}" iyz="0.0"
+                    izz="${(2/5) * mass * (radius*radius)}" />
+        </inertial>
+    </xacro:macro>
 </robot>

File: description/robot.body.xacro (robot description, xacro)
@@ -50,8 +50,10 @@
     <!-- Front Left Wheel -->
     <joint name="front_left_wheel_joint" type="continuous">
-        <parent link="chassis"/>
+        <parent link="base_link"/>
         <child link="front_left_wheel"/>
-        <origin xyz="0.29 0.175 0" rpy="-${pi/2} 0 0"/>
+        <origin xyz="0.2 0.175 0" rpy="-${pi/2} 0 0"/>
         <axis xyz="0 0 1"/>
+        <limit effort="1000" velocity="1000"/>
+        <dynamics damping="0.1" friction="0.2"/>
     </joint>
     <link name="front_left_wheel">
@@ -73,13 +75,15 @@
     <gazebo reference="front_left_wheel">
         <material>Gazebo/Black</material>
-        <mu1 value="0.0"/>
-        <mu2 value="0.0"/>
+ <!---     <mu1 value="0.0"/> -->
+  <!---    <mu2 value="0.0"/> -->
     </gazebo>
     <!-- Front Right Wheel -->
     <joint name="front_right_wheel_joint" type="continuous">
-        <parent link="chassis"/>
+        <parent link="base_link"/>
         <child link="front_right_wheel"/>
-        <origin xyz="0.29 -0.175 0" rpy="${pi/2} 0 0"/>
+        <origin xyz="0.2 -0.175 0" rpy="${pi/2} 0 0"/>
         <axis xyz="0 0 1"/>
+        <limit effort="1000" velocity="1000"/>
+        <dynamics damping="0.1" friction="0.2"/>
     </joint>
     <link name="front_right_wheel">
@@ -101,6 +105,6 @@
     <gazebo reference="front_right_wheel">
         <material>Gazebo/Black</material>
-        <mu1 value="0.0"/>
-        <mu2 value="0.0"/>
+ <!--       <mu1 value="0.0"/>  -->
+ <!--       <mu2 value="0.0"/>  -->
     </gazebo>
     <!-- Rear Left Wheel -->
@@ -108,6 +112,8 @@
         <parent link="base_link"/>
         <child link="rear_left_wheel"/>
-        <origin xyz="-0.15 0.175 0" rpy="-${pi/2} 0 0"/>
+        <origin xyz="-0.2 0.175 0" rpy="-${pi/2} 0 0"/>
         <axis xyz="0 0 1"/>
+        <limit effort="10000" velocity="1000" />
+	    <dynamics damping="1.0" friction="1.0" />
     </joint>
     <link name="rear_left_wheel">
@@ -134,6 +140,8 @@
         <parent link="base_link"/>
         <child link="rear_right_wheel"/>
-        <origin xyz="-0.15 -0.175 0" rpy="${pi/2} 0 0"/>
+        <origin xyz="-0.2 -0.175 0" rpy="${pi/2} 0 0"/>
         <axis xyz="0 0 1"/>
+		<limit effort="10000" velocity="1000" />
+	    <dynamics damping="1.0" friction="1.0" />
     </joint>
     <link name="rear_right_wheel">

Commit message: Working 4 wheel work, I need improvements in inertia

File: description/gazebo.control.xacro (robot description, xacro)
@@ -5,5 +5,5 @@
         <!-- Wheels-->
             <left_joint>front_left_wheel_joint</left_joint>
-            <left_joint>front_right_wheel_joint</left_joint>
+            <right_joint>front_right_wheel_joint</right_joint>
             <wheel_separation>0.35</wheel_separation>
             <wheel_diameter>0.1</wheel_diameter>
@@ -23,5 +23,5 @@
         <!-- Wheels-->
             <left_joint>rear_left_wheel_joint</left_joint>
-            <left_joint>rear_right_wheel_joint</left_joint>
+            <right_joint>rear_right_wheel_joint</right_joint>
             <wheel_separation>0.35</wheel_separation>
             <wheel_diameter>0.1</wheel_diameter>

File: description/inertial.macros.xacro (robot description, xacro)
@@ -21,12 +21,3 @@
         </inertial>
     </xacro:macro>
-    <xacro:macro name="inertial_sphere" params="mass radius *origin">
-        <inertial>
-            <xacro:insert_block name="origin"/>
-            <mass value="${mass}" />
-            <inertia ixx="${(2/5) * mass * (radius*radius)}" ixy="0.0" ixz="0.0"
-                    iyy="${(2/5) * mass * (radius*radius)}" iyz="0.0"
-                    izz="${(2/5) * mass * (radius*radius)}" />
-        </inertial>
-    </xacro:macro>
 </robot>

File: description/robot.body.xacro (robot description, xacro)
@@ -54,6 +54,4 @@
         <origin xyz="0.2 0.175 0" rpy="-${pi/2} 0 0"/>
         <axis xyz="0 0 1"/>
-        <limit effort="1000" velocity="1000"/>
-        <dynamics damping="0.1" friction="0.2"/>
     </joint>
     <link name="front_left_wheel">
@@ -84,6 +82,4 @@
         <origin xyz="0.2 -0.175 0" rpy="${pi/2} 0 0"/>
         <axis xyz="0 0 1"/>
-        <limit effort="1000" velocity="1000"/>
-        <dynamics damping="0.1" friction="0.2"/>
     </joint>
     <link name="front_right_wheel">
@@ -114,6 +110,4 @@
         <origin xyz="-0.2 0.175 0" rpy="-${pi/2} 0 0"/>
         <axis xyz="0 0 1"/>
-        <limit effort="10000" velocity="1000" />
-	    <dynamics damping="1.0" friction="1.0" />
     </joint>
     <link name="rear_left_wheel">
@@ -142,6 +136,4 @@
         <origin xyz="-0.2 -0.175 0" rpy="${pi/2} 0 0"/>
         <axis xyz="0 0 1"/>
-		<limit effort="10000" velocity="1000" />
-	    <dynamics damping="1.0" friction="1.0" />
     </joint>
     <link name="rear_right_wheel">

Commit message: Slam Toolbox added, evironment mapped

File: description/gazebo.control.xacro (robot description, xacro)
@@ -13,5 +13,5 @@
         <!-- Output-->
             <odometry_frame>odom</odometry_frame>
-            <robot_base_frame>base_link</robot_base_frame>
+            <robot_base_frame>base_footprint</robot_base_frame>
             <publish_odom>true</publish_odom>
             <publish_odom_tf>true</publish_odom_tf>
@@ -31,5 +31,5 @@
         <!-- Output-->
             <odometry_frame>odom</odometry_frame>
-            <robot_base_frame>base_link</robot_base_frame>
+            <robot_base_frame>base_footprint</robot_base_frame>
             <publish_odom>true</publish_odom>
             <publish_odom_tf>true</publish_odom_tf>

File: description/lidar.xacro (robot description, xacro)
@@ -1,13 +1,13 @@
 <?xml version="1.0"?>
-<robot xmlns:xacro="hhtp://www.ros.org/wiki/xacro" >
-    <joint name="lidar_joint" type="fixed">
+<robot xmlns:xacro="http://www.ros.org/wiki/xacro" >
+    <joint name="laser_joint" type="fixed">
         <parent link="chassis"/>
-        <child link="lidar_joint"/>
+        <child link="laser_frame"/>
         <origin xyz="0.1 0 0.175" rpy="0 0 0"/>
     </joint>
-    <link name="lidar_frame">
+    <link name="laser_frame">
         <visual>
             <geometry>
-                <cylinder radius="0.1" length="0.04"/>
+                <cylinder radius="0.05" length="0.04"/>
             </geometry>
             <material name="red"/>
@@ -15,10 +15,41 @@
         <collision>
             <geometry>
-                <cylinder radius="0.1" length="0.04"/>
+                <cylinder radius="0.05" length="0.04"/>
             </geometry>
         </collision>
-        <xacro:inertial_cylinder mass="0.1" length="0.04" radius="0.1">
+        <xacro:inertial_cylinder mass="0.1" length="0.04" radius="0.05">
             <origin xyz="0 0 0" rpy="0 0 0"/>
         </xacro:inertial_cylinder>
     </link>
+    <gazebo reference="laser_frame">
+        <material>Gazebo/Red</material>
+        <sensor name="laser" type="ray">
+            <pose> 0 0 0 0 0 0 </pose>
+            <visualize>true</visualize>
+            <always_on>true</always_on>
+            <update_rate>10</update_rate>
+            <ray>
+                <scan>
+                    <horizontal>
+                        <samples>360</samples>
+                        <resolution>1</resolution>
+                        <min_angle>-3.14</min_angle>
+                        <max_angle>3.14</max_angle>
+                    </horizontal>
+                </scan>
+                <range>
+                    <min>0.3</min>
+                    <max>12</max>
+                    <resolution>0.01</resolution>
+                </range>
+            </ray>
+            <plugin name="laser_controller" filename="libgazebo_ros_ray_sensor.so">
+                <ros>
+                    <remapping>~/out:=scan</remapping>
+                </ros>
+                <output_type>sensor_msgs/LaserScan</output_type>
+                <frame_name>laser_frame</frame_name>
+            </plugin>
+        </sensor>
+    </gazebo>
 </robot>

File: description/robot.body.xacro (robot description, xacro)
@@ -18,7 +18,15 @@
         <color rgba="1 0 0 1"/>
     </material>
+    <!-- Base Footprint -->
+    <link name="base_footprint"/>
     <!-- Base Link -->
     <link name="base_link">
     </link>
+    <!-- Base Footprint -->
+    <joint name="base_footprint_joint" type="fixed">
+        <parent link="base_footprint"/>
+        <child link="base_link"/>
+        <origin xyz="0 0 0"/>
+    </joint>
     <!-- Chassis -->
     <joint name="chassis_joint" type="fixed">

File: description/robot.urdf.xacro (robot description, xacro)
@@ -3,3 +3,4 @@
     <xacro:include filename="robot.body.xacro" />
     <xacro:include filename="gazebo.control.xacro"/>
+    <xacro:include filename="lidar.xacro"/>
 </robot>
